File: MSPY.kicad_pcb (KiCad board)
At the start: 2 copper layers, 15.7 x 43.4 mm, 13 parts, among them J1 Conn_01x06, J2 Conn_01x12, J3 Conn_01x12, SW1 SW_Push, U1 MSP430FR2433RGE

Commit message: WIP
Parts:
- moved U1 3.94 mm to (153.7, 92.6)
Routing:
- net P12: track 10.4 -> 0.00 mm
- net P11: track 10.3 -> 0.00 mm
- net P16: track 43.4 -> 33.2 mm
- net P10: track 8.64 -> 0.00 mm
- net P9: track 7.70 -> 0.00 mm
- net P8: track 7.21 -> 0.00 mm
- net P13: track 6.05 -> 0.00 mm
- net VCC: track 27.8 -> 23.2 mm
- net P15: track 4.36 -> 0.00 mm
- net P7: track 7.93 -> 3.64 mm
- net P14: track 5.21 -> 1.70 mm
- net P6: track 8.85 -> 5.99 mm
- net P3: track 35.3 -> 32.8 mm
- net VSS: track 41.8 -> 39.4 mm, vias 2 -> 1
- net P17: track 32.0 -> 29.9 mm
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Other:
- board text removed: "MSPY"
- board text removed: "birchavenue.org"
- board text removed: "v1.1"

Commit message: WIP
Parts:
- added C4: 33 pF, Capacitor_SMD:C_0603_1608Metric_Pad1.08x0.95mm_HandSolder, F.Cu at (152.5, 85.1)
- added C5: 33 pf, Capacitor_SMD:C_0603_1608Metric_Pad1.08x0.95mm_HandSolder, F.Cu at (155.5, 82.6)
- added R6: 0, Resistor_SMD:R_0603_1608Metric_Pad0.98x0.95mm_HandSolder, F.Cu at (150.9, 85.1)
- added R7: 0, Resistor_SMD:R_0603_1608Metric_Pad0.98x0.95mm_HandSolder, F.Cu at (155.5, 80.9)
- added Y1: Crystal_GND24, Crystal:Crystal_SMD_SeikoEpson_TSX3225-4Pin_3.2x2.5mm, F.Cu at (155.5, 85.1)
- C1, C2, C3: footprint Capacitor_SMD:C_0603_1608Metric_Pad1.05x0.95mm_HandSolder -> Capacitor_SMD:C_0603_1608Metric_Pad1.08x0.95mm_HandSolder
- moved C1 15.7 mm to (171.5, 84.7)
- moved C2 15.5 mm to (169.9, 84.7)
- moved C3 15.4 mm to (167.3, 85.5)
- moved R5 15.4 mm to (167.3, 83.9)
- moved U1 0.28 mm to (153.4, 92.7), turned to -45 degrees
Connections:
- U1 pad 21: P21 -> XOUT
- U1 pad 22: P22 -> XIN
- U1 pad 25: (no net) -> VSS
Routing:
- net P3: track 32.8 -> 0.00 mm, vias 1 -> 0
- net P16: track 33.2 -> 4.79 mm, vias 1 -> 0
- net P4: track 27.5 -> 0.00 mm
- net VSS: track 39.4 -> 12.5 mm, vias 1 -> 0
- net P17: track 29.9 -> 7.28 mm
- net P22: track 18.7 -> 0.00 mm
- net P21: track 16.5 -> 0.00 mm
- net VCC: track 23.2 -> 6.85 mm
- net P2: track 14.7 -> 0.00 mm
- net P20: track 12.7 -> 0.00 mm
- net P1: track 19.1 -> 8.09 mm
- net P19: track 10.2 -> 0.00 mm
- net P5: track 9.43 -> 0.00 mm
- net P6: track 5.99 -> 0.00 mm
- net XOUT: track 0.00 -> 5.67 mm
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