File: MSPY.kicad_sch (KiCad schematic)
At the start: 13 parts, among them J1 Conn_01x06, J2 Conn_01x12, J3 Conn_01x12, SW1 SW_Push, U1 MSP430FR2433RGE

Commit message: WIP
Parts:
- added C1: 33 pF, Capacitor_SMD:C_0603_1608Metric_Pad1.05x0.95mm_HandSolder, symbol Device:C
- added C3: 33 pf, Capacitor_SMD:C_0603_1608Metric_Pad1.05x0.95mm_HandSolder, symbol Device:C
- added R5, R6: 0, Resistor_SMD:R_0603_1608Metric_Pad0.98x0.95mm_HandSolder, symbol Device:R
- added Y1: Crystal_GND24, Crystal:Crystal_SMD_SeikoEpson_TSX3225-4Pin_3.2x2.5mm, symbol Device:Crystal_GND24
- renumbered C1 to C2, C2 to C4, C3 to C5, R5 to R7
Connections:
- net P21: now also R6.1; no longer U1.21 (P2.0/XOUT)
- net P22: now also R5.1; no longer U1.22 (P2.1/XIN)
- net VSS: now also C1.2, C3.2, Y1.2, Y1.4
- new net XIN: C1.1, R5.2, U1.22 (P2.1/XIN), Y1.1
- new net XOUT: C3.1, R6.2, U1.21 (P2.0/XOUT), Y1.3

Commit message: WIP
Parts:
- removed U1: MSP430FR2433RGE, Package_DFN_QFN:VQFN-24-1EP_4x4mm_P0.5mm_EP2.45x2.45mm, symbol MSPY-rescue:MSP430FR2433RGE-extended
- added U1: MSP430FR2433RGE, Package_DFN_QFN:VQFN-24-1EP_4x4mm_P0.5mm_EP2.45x2.45mm, symbol extended:MSP430FR2433RGE
- C1: renamed from C2; footprint Capacitor_SMD:C_0603_1608Metric_Pad1.05x0.95mm_HandSolder -> Capacitor_SMD:C_0603_1608Metric_Pad1.08x0.95mm_HandSolder
- C2: renamed from C4; footprint Capacitor_SMD:C_0603_1608Metric_Pad1.05x0.95mm_HandSolder -> Capacitor_SMD:C_0603_1608Metric_Pad1.08x0.95mm_HandSolder
- C3: renamed from C5; footprint Capacitor_SMD:C_0603_1608Metric_Pad1.05x0.95mm_HandSolder -> Capacitor_SMD:C_0603_1608Metric_Pad1.08x0.95mm_HandSolder
- C4: renamed from C1; footprint Capacitor_SMD:C_0603_1608Metric_Pad1.05x0.95mm_HandSolder -> Capacitor_SMD:C_0603_1608Metric_Pad1.08x0.95mm_HandSolder
- C5: renamed from C3; footprint Capacitor_SMD:C_0603_1608Metric_Pad1.05x0.95mm_HandSolder -> Capacitor_SMD:C_0603_1608Metric_Pad1.08x0.95mm_HandSolder
- renumbered R7 to R1, R1 to R2, R2 to R3, R3 to R4, R4 to R5, R5 to R6, R6 to R7
Connections:
- net P1: now also U1.1 (RST/NMI/SBWTDIO)
- net P10: now also U1.10 (P1.3/UCB0SOMI/UCB0SCL/MCLK/A3)
- net P11: now also U1.11 (P2.2/ACLK)
- net P12: now also U1.12 (P3.0)
- net P13: now also U1.13 (P2.3)
- net P14: now also U1.14 (P3.1/UCA1STE)
- net P15: now also U1.15 (P2.4/UCA1CLK)
- net P16: now also U1.16 (P2.5/UCA1RXD/UCA1SOMI)
- net P17: now also U1.17 (P2.6/UCA1TXD/UCA1SIMO)
- net P19: now also U1.19 (P2.7)
- net P2: now also U1.2 (TEST/SBWTCK)
- net P20: now also U1.20 (P3.2)
- net P3: now also U1.3 (P1.4/UCA0TXD/UCA0SIMO/TA1.2/TCK/A4/VREF+)
- net P4: now also U1.4 (P1.5/UCA0RXD/UCA0SOMI/TA1.1/TMS/A5)
- net P5: now also U1.5 (P1.6/UCA0CLK/TA1CLK/TDI/TCLK/A6)
- net P6: now also U1.6 (P1.7/UCA0STE/SMCLK/TDO/A7)
- net P7: now also U1.7 (P1.0/UCB0STE/TA0CLK/A0/Veref+)
- net P8: now also U1.8 (P1.1/UCB0CLK/TA0.1/A1)
- net P9: now also U1.9 (P1.2/UCB0SIMO/UCB0SDA/TA0.2/A2/Veref)
- net VCC: now also U1.24 (DVCC)
- net VSS: now also U1.18 (DVSS), U1.23 (DVSS), U1.25 (VSS)
- net XIN: now also U1.22 (P2.1/XIN)
- net XOUT: now also U1.21 (P2.0/XOUT)
Other:
- moved on the sheet: C1, C2, C3, R1, SW1
